File: Eagle-Board/bike_tracker.brd (EAGLE design)
At the start: 70 x 33 mm, 69 parts, among them J1 TRANSFLASH-LOCK, Q1 IRLML5203, Q2 IRLML5203, Q3 IRLML5203, Q4 IRLML5203

Commit message: revision v1.2
Parts:
- removed JP2: (no value), pinhead:1X04
- removed R25, R26, R27: (no value), resistor:R0201
- removed U$2: GPS-NEO6M, diy-modules:GPS-RECEIVER-NEO6M2
- removed U$3: MPU9255, diy-modules:MPU9255
- removed U$4: BME280, diy-modules:BME280
- added BAT1: XH414, microduino:TS414H
- added C1: 10uF, microduino:EIA3528
- added C10, C11: 0.1uF, SparkFun-Capacitors:0603
- added C7: 0.1uF, microduino:0603-CAP
- added C8, C9: 0.1uF, SparkFun-Capacitors:0603-CAP
- added D1: MBR0520, microduino:SOD123
- added IC1: 24C00TS, microchip:TSSOP8
- added IC2: BME280, bosch-bme280:BME280
- added IPEX: ANT-UMCC, microduino:UMCC
- added JP3: JUMPER-SMT_3_1-NC_TRACE_NO-SILK, SparkFun-Jumpers:SMT-JUMPER_3_1-NC_TRACE_NO-SILK
- added L1: (no value), microduino:0603
- added R30, R31, R33: 1k, microduino:0603-RES
- added R32: null, microduino:0603-RES
- added R34: 10, microduino:0603-RES
- added R35, R36, R37: 10K, SparkFun-Resistors:0603-RES
- added R40, R41: 4.7k, SparkFun-Resistors:0603
- added R42: (no value), resistor:R0201
- added SJ2: JUMPER_PAD-3-1&2_NC_BY_PASTE, SparkFun-Passives:PAD-HUMPER-3-1&2_NC_BY_PASTE_YES_SILK_FULL_BOX
- added STATUS: green, microduino:0805-LED
- added U$6: BLOX-NEO-6M, microduino:NE0-6M
- added U1: MPU-9250, Testing:QFN24_PAD
- moved R24 132.7 mm to (-44.1, -31.0), turned to 0 degrees
Connections:
- new net !CS: R37.1, U1.22
- new net AD0/SDO: SJ2.3
- new net ADSD_STUB: SJ2.2, U1.9
- new net AUX_CL: U1.7
- new net AUX_DA: U1.21
- new net FSYNC: U1.11
- new net N$16: R30.2, STATUS.A
- new net N$17: STATUS.C, U$6.3
- new net N$18: IPEX.3, L1.1, U$6.11
- new net N$19: R31.1, U$6.21
- new net N$20: R32.1, U$6.15
- new net N$21: R33.1, U$6.14
- new net N$22: BAT1.1, D1.C, U$6.22
- new net N$23: L1.2, R34.2
- new net N$24: R34.1, U$6.8, U$6.9
- new net N$25: IC2.2, R40.1
- new net N$26: JP3.1, R41.1
- new net REGOUT: C8.1, U1.10
- new net RXD-NEO: R31.2
- new net SCL_GPS: IC1.6, U$6.19
- new net SDA_GPS: IC1.5, U$6.18
- new net SDO: IC2.5, JP3.2
- new net VDDIO: R35.2, R36.2, R37.2, U1.1, U1.8
- net GND: now also C9.2, R42.2, SJ2.1; no longer R25.1, R26.1, R27.1
- net GND_BME: now also C10.2, C11.2, IC2.1, IC2.7, JP3.3, R24.2; no longer R26.2, U$4.2
- net GND_GPS: now also BAT1.2, C1.C, C7.2, IC1.4, IPEX.1, IPEX.2, R32.2, R33.2, U$6.10, U$6.12, U$6.13, U$6.24, U$6.7; no longer JP2.1, R24.2, R27.2, U$2.4
- net GND_MPU: now also C8.2, R42.1, U1.18, U1.20, U1.CENTER; no longer R25.2, U$3.2
- net INT-IMU: now also U1.12; no longer U$3.8
- net RXD_NEO: no longer JP2.3, U$2.3
- net SCL-BME: now also IC2.4; no longer U$4.3
- net SCL-IMU: now also R36.1, U1.23; no longer U$3.3
- net SDA-BME: now also IC2.3; no longer U$4.4
- net SDA-IMU: now also R35.1, U1.24; no longer U$3.4
- net TXD-NEO: now also U$6.20; no longer JP2.2, U$2.2
- net VDD: now also C1.A, C10.1, C11.1, C7.1, C9.1, D1.A, IC1.8, IC2.6, IC2.8, R30.1, R40.2, R41.2, U$6.23, U1.13; no longer JP2.4, U$2.1, U$3.1, U$4.1
Routing:
- net GND_GPS: track 24.5 -> 0.02 mm, vias 1 -> 0
- net VDD: track 169.5 -> 145.8 mm
- net TXD-NEO: track 18.0 -> 9.50 mm
- net RXD_NEO: track 11.0 -> 3.32 mm
- net N$3: track 14.9 -> 7.67 mm
- net GND_BME: track 13.3 -> 8.81 mm
- net GND_MPU: track 14.0 -> 11.1 mm
- net INT-IMU: track 18.2 -> 15.8 mm
- net N$1: track 15.5 -> 13.2 mm
- net SDA-BME: track 9.31 -> 7.41 mm
- net SDA-IMU: track 17.3 -> 16.1 mm
- net SCL-IMU: track 19.0 -> 17.8 mm
- net N$2: track 23.4 -> 22.4 mm
- net SCL-BME: track 14.9 -> 14.0 mm

Commit message: first commit rev1.2
Parts:
- removed R37: 10K, SparkFun-Resistors:0603-RES
- moved R24 135.3 mm to (58.8, 56.9)
- moved C10 117.6 mm to (66.8, 55.2)
- moved C11 115.6 mm to (66.8, 56.5)
- moved R42 112.6 mm to (15.0, 68.5), flipped to the bottom
- moved R40 112.2 mm to (62.5, 48.8), turned to 180 degrees
- moved R41 110.2 mm to (62.5, 50.0), flipped to the bottom
- moved JP3 106.7 mm to (63.4, 54.4), turned to 90 degrees
- moved IC2 101.4 mm to (66.3, 52.2)
- moved R35 79.9 mm to (24.3, 69.1), flipped to the bottom, turned to 180 degrees
- moved R36 79.0 mm to (24.3, 70.4), flipped to the bottom, turned to 180 degrees
- moved C9 76.3 mm to (17.5, 67.9), flipped to the bottom, turned to 90 degrees
- moved SJ2 75.1 mm to (25.0, 66.4), flipped to the bottom
- moved C8 74.6 mm to (17.5, 64.1), flipped to the bottom
- moved U1 68.3 mm to (20.8, 66.8), flipped to the bottom
- moved L1 58.7 mm to (46.9, 62.7), turned to 270 degrees
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Connections:
- removed net !CS: R37.1, U1.22
- removed net RXD_NEO: SH8.1
- net GND: no longer C9.2, SJ2.1
- net GND_MPU: now also C9.2, SJ2.1
- net RXD-NEO: now also SH8.1
- net VDDIO: no longer R37.2
Routing:
- net VDD: track 145.8 -> 212.3 mm, vias 3 -> 11
- net N$18: track 0.00 -> 29.6 mm, vias 0 -> 1
- net VBAT-: track 45.1 -> 20.7 mm
- net N$19: track 0.00 -> 20.2 mm, vias 0 -> 3
- net VBAT+: track 47.7 -> 29.5 mm
- net N$22: track 0.00 -> 17.2 mm, vias 0 -> 1
- net IO32: track 21.8 -> 10.7 mm
- net VDDIO: track 0.00 -> 10.3 mm
- net N$21: track 0.00 -> 7.69 mm, vias 0 -> 1
- net N$3: track 7.67 -> 15.1 mm
- net TXD-NEO: track 9.50 -> 2.44 mm
- net ADSD_STUB: track 0.00 -> 6.90 mm
- net INT-IMU: track 15.8 -> 9.48 mm, vias 0 -> 1
- net GND: track 2.12 -> 8.41 mm, vias 37 -> 31
- net N$24: track 0.00 -> 5.78 mm, vias 0 -> 1
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- added copper zone on layer 1, net GND_BME
- added copper zone on layer 16, net GND_BME
- added copper zone on layer 1, net GND_GPS
- added copper zone on layer 16, net GND_GPS
- added copper zone on layer 16, net GND_MPU
Other:
- board text added: "BikeTracker V1.2"
- board text added: "X"
- board text added: "Y"
- board text added: "Z"
- board text removed: "BikeTracker V1.1"

Commit message: minor modifications
Parts:
- moved SH10 1.92 mm to (55.1, 51.9)
- moved C3 0.92 mm to (23.7, 55.9)
- moved C6 0.74 mm to (24.4, 57.8)
- moved R11 0.68 mm to (29.6, 55.1)
Routing:
- net SDA: track 51.9 -> 49.8 mm
- net SDA-BME: track 10.7 -> 12.7 mm
- net VBAT+: track 29.5 -> 28.5 mm
- net VBAT-: track 20.7 -> 19.9 mm
- net N$14: track 8.55 -> 7.91 mm
Changed lines of the file:
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@@
 <attribute name="NAME" x="16.764" y="60.198" size="0.508" layer="25" font="vector" ratio="15" rot="R90"/>
 </element>
-<element name="C3" library="rcl" package="C0603" value="0.47u" x="24.003" y="54.991" smashed="yes">
-<attribute name="NAME" x="22.86" y="55.753" size="0.508" layer="25" font="vector" ratio="15"/>
+<element name="C3" library="rcl" package="C0603" value="0.47u" x="23.749" y="55.88" smashed="yes">
+<attribute name="NAME" x="22.606" y="56.642" size="0.508" layer="25" font="vector" ratio="15"/>
 </element>
 <element name="C4" library="rcl" package="C0603" value="0.1u" x="27.94" y="58.674" smashed="yes" rot="R270">
@@
 <attribute name="NAME" x="31.877" y="57.277" size="0.508" layer="25" font="vector" ratio="15" rot="R90"/>
 </element>
-<element name="C6" library="rcl" package="C0603" value="0.1u" x="23.749" y="58.166" smashed="yes">
-<attribute name="NAME" x="22.479" y="58.801" size="0.508" layer="25" font="vector" ratio="15"/>
+<element name="C6" library="rcl" package="C0603" value="0.1u" x="24.384" y="57.785" smashed="yes">
+<attribute name="NAME" x="23.114" y="58.42" size="0.508" layer="25" font="vector" ratio="15"/>
 </element>
 <element name="J1" library="sd-mmc" package="TRANSFLASH-LOCK-SOCK" value="TRANSFLASH-LOCK" x="67.31" y="66.675" smashed="yes">
@@
 <attribute name="NAME" x="31.0515" y="63.119" size="0.508" layer="25" font="vector" ratio="15" rot="R180"/>
 </element>
-<element name="R11" library="resistor" package="R0603" value="0.01" x="30.226" y="55.372" smashed="yes" rot="R90">
-<attribute name="NAME" x="31.75" y="55.245" size="0.508" layer="25" font="vector" ratio="15" rot="R90"/>
+<element name="R11" library="resistor" package="R0603" value="0.01" x="29.591" y="55.118" smashed="yes" rot="R90">
+<attribute name="NAME" x="30.861" y="55.245" size="0.508" layer="25" font="vector" ratio="15" rot="R90"/>
 </element>
 <element name="R12" library="resistor" package="R0603" value="100" x="27.432" y="55.88" smashed="yes">
@@
 <element name="SH8" library="shorts" package="SHORT_TOP-20" value="SHORT" x="48.895" y="55.88" smashed="yes" rot="R180"/>
 <element name="SH9" library="shorts" package="SHORT_TOP-20" value="SHORT" x="53.213" y="53.594" smashed="yes" rot="MR180"/>
-<element name="SH10" library="shorts" package="SHORT_TOP-20" value="SHORT" x="57.023" y="51.689" smashed="yes"/>
+<element name="SH10" library="shorts" package="SHORT_TOP-20" value="SHORT" x="55.118" y="51.943" smashed="yes"/>
 <element name="BAT-IN" library="con-garry" library_urn="urn:adsk.eagle:library:147" package="332-02" package3d_urn="urn:adsk.eagle:package:6810/1" value="332-02" x="14.097" y="56.515" smashed="yes" rot="R90">
 <attribute name="NAME" x="16.256" y="55.387" size="0.508" layer="26" font="vector" ratio="15" rot="MR90"/>
@@
 </element>
 <element name="R20" library="ssmd" package="0603" value="10k" x="55.626" y="53.086" smashed="yes" rot="R180">
-<attribute name="NAME" x="55.753" y="52.324" size="0.508" layer="25" font="vector" ratio="15" rot="R180"/>
+<attribute name="NAME" x="56.642" y="54.102" size="0.508" layer="25" font="vector" ratio="15" rot="R180"/>
 </element>
 <element name="R21" library="ssmd" package="0603" value="470R" x="54.102" y="55.88" smashed="yes" rot="R180">
@@
 <via x="19.939" y="61.4172" extent="1-16" drill="0.35"/>
 <wire x1="19.939" y1="61.4172" x2="18.796" y2="60.2742" width="0.254" layer="16"/>
-<wire x1="23.153" y1="54.991" x2="21.971" y2="56.173" width="0.254" layer="1"/>
+<wire x1="22.899" y1="55.88" x2="21.971" y2="56.808" width="0.254" layer="1"/>
 <wire x1="21.971" y1="57.785" x2="21.209" y2="58.547" width="0.254" layer="1"/>
-<wire x1="21.971" y1="57.785" x2="21.971" y2="56.173" width="0.254" layer="1"/>
+<wire x1="21.971" y1="57.785" x2="21.971" y2="56.808" width="0.254" layer="1"/>
 <contactref element="BAT-IN" pad="2"/>
 <contactref element="BAT" pad="1"/>
@@
 <wire x1="26.146" y1="60.214" x2="26.543" y2="59.817" width="0.254" layer="1"/>
 <wire x1="25.47" y1="60.214" x2="26.146" y2="60.214" width="0.254" layer="1"/>
-<wire x1="26.543" y1="59.817" x2="26.543" y2="58.166" width="0.254" layer="1"/>
-<wire x1="26.543" y1="58.166" x2="26.543" y2="57.785" width="0.254" layer="1"/>
+<wire x1="26.543" y1="59.817" x2="26.543" y2="57.785" width="0.254" layer="1"/>
 <wire x1="26.543" y1="57.785" x2="26.543" y2="55.919" width="0.254" layer="1"/>
 <wire x1="26.543" y1="55.919" x2="26.582" y2="55.88" width="0.254" layer="1"/>
 <wire x1="27.94" y1="57.824" x2="26.582" y2="57.824" width="0.254" layer="1"/>
 <wire x1="26.582" y1="57.824" x2="26.543" y2="57.785" width="0.254" layer="1"/>
-<wire x1="26.543" y1="58.166" x2="24.599" y2="58.166" width="0.254" layer="1"/>
+<wire x1="26.543" y1="57.785" x2="25.234" y2="57.785" width="0.254" layer="1"/>
 </signal>
 <signal name="N$11">
@@
 <contactref element="BAT" pad="2"/>
 <wire x1="18.796" y1="54.991" x2="18.796" y2="56.531" width="0.254" layer="1"/>
-<wire x1="30.226" y1="56.222" x2="28.624" y2="56.222" width="0.254" layer="1"/>
-<wire x1="28.282" y1="55.88" x2="28.624" y2="56.222" width="0.254" layer="1"/>
+<wire x1="29.591" y1="55.968" x2="28.37" y2="55.968" width="0.254" layer="1"/>
+<wire x1="28.282" y1="55.88" x2="28.37" y2="55.968" width="0.254" layer="1"/>
 <wire x1="18.796" y1="56.531" x2="17.145" y2="56.531" width="0.508" layer="16"/>
 <wire x1="17.145" y1="56.531" x2="16.907" y2="56.531" width="0.508" layer="16"/>
@@
 <wire x1="65.969" y1="50.094" x2="65.532" y2="49.657" width="0.254" layer="1"/>
 <wire x1="61.976" y1="49.657" x2="65.532" y2="49.657" width="0.254" layer="1"/>
-<wire x1="57.404" y1="51.689" x2="59.944" y2="51.689" width="0.254" layer="1"/>
-<wire x1="59.944" y1="51.689" x2="61.976" y2="49.657" width="0.254" layer="1"/>
+<wire x1="55.499" y1="51.943" x2="59.69" y2="51.943" width="0.254" layer="1"/>
+<wire x1="59.69" y1="51.943" x2="61.976" y2="49.657" width="0.254" layer="1"/>
 </signal>
 <signal name="TXD-NEO">
@@
 <contactref element="SH3" pad="2"/>
 <contactref element="SH10" pad="2"/>
-<wire x1="48.26" y1="51.689" x2="47.879" y2="52.07" width="0.254" layer="1"/>
+<wire x1="48.26" y1="51.689" x2="47.117" y2="52.832" width="0.254" layer="1"/>
 <wire x1="48.26" y1="51.689" x2="48.26" y2="50.185" width="0.254" layer="1"/>
 <wire x1="48.26" y1="50.185" x2="48.25" y2="50.175" width="0.254" layer="1"/>
 <wire x1="33.274" y1="60.198" x2="32.639" y2="60.198" width="0.254" layer="1"/>
-<via x="52.832" y="52.07" extent="1-16" drill="0.35"/>
-<wire x1="52.832" y1="52.07" x2="48.641" y2="52.07" width="0.254" layer="16"/>
+<via x="52.959" y="51.943" extent="1-16" drill="0.35"/>
+<wire x1="52.959" y1="51.943" x2="48.514" y2="51.943" width="0.254" layer="16"/>
 <wire x1="48.25" y1="51.679" x2="48.25" y2="50.175" width="0.254" layer="16"/>
-<wire x1="48.641" y1="52.07" x2="48.25" y2="51.679" width="0.254" layer="16"/>
-<wire x1="34.036" y1="52.07" x2="47.879" y2="52.07" width="0.254" layer="1"/>
+<wire x1="48.514" y1="51.943" x2="48.25" y2="51.679" width="0.254" layer="16"/>
+<wire x1="33.274" y1="52.832" x2="47.117" y2="52.832" width="0.254" layer="1"/>
 <contactref element="R9" pad="2"/>
 <contactref element="SH11" pad="2"/>
@@
 <wire x1="53.594" y1="61.341" x2="53.213" y2="61.341" width="0.254" layer="1"/>
 <wire x1="53.213" y1="61.341" x2="52.07" y2="60.198" width="0.254" layer="1"/>
-<wire x1="56.896" y1="51.689" x2="53.213" y2="51.689" width="0.254" layer="1"/>
-<wire x1="53.213" y1="51.689" x2="52.832" y2="52.07" width="0.254" layer="1"/>
+<wire x1="54.991" y1="51.943" x2="52.959" y2="51.943" width="0.254" layer="1"/>
 <wire x1="49.403" y1="54.864" x2="48.26" y2="54.864" width="0.254" layer="1"/>
 <wire x1="46.863" y1="56.261" x2="46.863" y2="57.062" width="0.254" layer="1"/>
 <wire x1="48.26" y1="54.864" x2="46.863" y2="56.261" width="0.254" layer="1"/>
 <wire x1="33.274" y1="60.198" x2="33.147" y2="60.071" width="0.254" layer="1"/>
-<wire x1="34.036" y1="52.07" x2="32.639" y2="53.467" width="0.254" layer="1"/>
+<wire x1="33.274" y1="52.832" x2="32.639" y2="53.467" width="0.254" layer="1"/>
 <wire x1="32.639" y1="53.467" x2="32.639" y2="60.198" width="0.254" layer="1"/>
 <wire x1="32.131" y1="60.198" x2="32.639" y2="60.198" width="0.254" layer="1"/>
@@
 <wire x1="49.5935" y1="64.0715" x2="50.673" y2="62.992" width="0.254" layer="1"/>
 <wire x1="36.957" y1="65.532" x2="36.957" y2="64.77" width="0.254" layer="1"/>
-<wire x1="43.17" y1="52.06" x2="43.815" y2="52.705" width="0.254" layer="16"/>
-<wire x1="43.815" y1="52.705" x2="52.07" y2="52.705" width="0.254" layer="16"/>
-<wire x1="52.07" y1="52.705" x2="52.578" y2="53.213" width="0.254" layer="16"/>
+<wire x1="43.17" y1="52.06" x2="43.942" y2="52.832" width="0.254" layer="16"/>
+<wire x1="43.942" y1="52.832" x2="52.197" y2="52.832" width="0.254" layer="16"/>
+<wire x1="52.197" y1="52.832" x2="52.578" y2="53.213" width="0.254" layer="16"/>
 <wire x1="49.657" y1="66.294" x2="49.657" y2="64.135" width="0.254" layer="16"/>
 <wire x1="49.657" y1="64.135" x2="49.5935" y2="64.0715" width="0.254" layer="16"/>

Commit message: modified and cleaned for production
Parts:
- added R25, R26, R27, R37: (no value), resistor:R0201
- C7: device microduino:0603-CAP -> rcl:R0603
- C8, C9: device SparkFun-Capacitors:0603-CAP -> resistor:C0603K
- IC2: value BME280 -> BME280/680
- R18, R19, R22, R23, R87, R90: device ssmd:0603 -> resistor:R0603
- R20, R21: device ssmd:0603 -> rcl:R0603
- R30: device microduino:0603-RES -> resistor:R0603
- R31, R32, R33, R34: device microduino:0603-RES -> rcl:R0603
- R35, R36: device SparkFun-Resistors:0603-RES -> resistor:R0603
- U1: value MPU-9250 -> MPU-9250/5; device Testing:QFN24_PAD -> invensense:LEAD-QFN24
- moved R41 0.97 mm to (62.4, 51.0)
- moved R2 0.89 mm to (56.5, 62.1)
- moved SH10 0.68 mm to (55.8, 51.7)
- moved SH9 0.38 mm to (53.3, 53.2)
- moved D1 0.35 mm to (43.5, 61.9)
- moved Q4 0.20 mm to (46.3, 67.5)
- moved Q5 0.20 mm to (56.2, 69.0), flipped to the bottom
- moved SH4 0.20 mm to (33.1, 60.3)
- moved R36 0.20 mm to (24.1, 70.5)
- moved R8 0.18 mm to (60.8, 60.1)
- moved R24 0.15 mm to (58.6, 56.9)
- moved Q1 0.15 mm to (55.8, 66.0)
- moved R90 0.15 mm to (47.7, 69.7)
- moved R35 0.13 mm to (24.1, 69.1)
- moved C9 0.10 mm to (17.4, 67.9)
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- renumbered STATUS to GPS-STATUS, U$6 to NEO-GPS
Connections:
- net ADSD_STUB renamed N$27
- net GND: now also R37.2
- net GND_GPS: now also R37.1
- net GND_MPU: now also U1.25; no longer U1.20, U1.CENTER
- net N$10: now also U$1.2; no longer U$1.1
- net N$13: now also U$1.1; no longer U$1.2
- net SCL: now also R27.2
- net SCL_GPS: now also R27.1
- net SDA: now also R26.2
- net SDA_GPS: now also R26.1
- net VDD: now also R25.1
- net VDDIO: now also R25.2
Routing:
- net GND: track 8.41 -> 26.6 mm, vias 31 -> 43
- net SCL: track 43.6 -> 53.1 mm, vias 2 -> 3
- net N$13: track 4.34 -> 9.14 mm
- net N$10: track 7.99 -> 4.95 mm
- net VDD: track 212.3 -> 215.3 mm, vias 11 -> 12
- net N$19: track 20.2 -> 23.2 mm
- net GND_BME: track 11.3 -> 8.45 mm
- net GND_MPU: track 7.95 -> 10.2 mm, vias 0 -> 4
- net SDA: track 49.8 -> 52.0 mm
- net VBAT-: track 19.9 -> 18.0 mm
- net SCL_GPS: track 3.81 -> 5.43 mm
- net SDA_GPS: track 5.45 -> 6.99 mm
- net IO32: track 10.7 -> 12.2 mm
- net SDO: track 3.95 -> 2.91 mm
- net VDDIO: track 10.3 -> 11.4 mm
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- added copper zone on layer 1, net GND_MPU
