File: Eagle-Board/bike_tracker.sch (EAGLE design)
At the start: 93 parts, among them IC1 24C00TS, IC2 BME280/680, J1 TRANSFLASH-LOCK, Q1 IRLML5203, Q2 IRLML5203, Q3 IRLML5203, Q4 IRLML5203, U1 MPU-9250/5

Commit message: minor modifications
Other:
- moved on the sheet: C7
Changed lines of the file:
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@@
 <attribute name="VALUE" x="336.296" y="33.909" size="1.778" layer="96"/>
 </instance>
-<instance part="C7" gate="G$1" x="342.9" y="35.56" smashed="yes">
-<attribute name="NAME" x="344.424" y="38.481" size="1.778" layer="95"/>
-<attribute name="VALUE" x="344.424" y="33.401" size="1.778" layer="96"/>
+<instance part="C7" gate="G$1" x="342.9" y="38.1" smashed="yes" rot="R270">
+<attribute name="NAME" x="345.821" y="36.576" size="1.778" layer="95" rot="R270"/>
+<attribute name="VALUE" x="340.741" y="36.576" size="1.778" layer="96" rot="R270"/>
 </instance>
 <instance part="IPEX" gate="G$1" x="220.98" y="12.7" smashed="yes"/>
@@
 <pinref part="J1" gate="G$1" pin="VDD"/>
 <pinref part="VDD2" gate="G$1" pin="VDD"/>
-<wire x1="60.96" y1="-38.1" x2="55.88" y2="-30.48" width="0.1524" layer="91"/>
+<wire x1="60.96" y1="-38.1" x2="55.88" y2="-38.1" width="0.1524" layer="91"/>
+<wire x1="55.88" y1="-38.1" x2="55.88" y2="-30.48" width="0.1524" layer="91"/>
 </segment>
 <segment>
@@
 <pinref part="C7" gate="G$1" pin="1"/>
 <wire x1="335.28" y1="43.18" x2="342.9" y2="43.18" width="0.1524" layer="91"/>
-<wire x1="342.9" y1="43.18" x2="337.82" y2="35.56" width="0.1524" layer="91"/>
 <junction x="335.28" y="43.18"/>
 <junction x="332.74" y="43.18"/>
@@
 <wire x1="335.28" y1="30.48" x2="342.9" y2="30.48" width="0.1524" layer="91"/>
 <pinref part="C7" gate="G$1" pin="2"/>
-<wire x1="342.9" y1="30.48" x2="347.98" y2="35.56" width="0.1524" layer="91"/>
+<wire x1="342.9" y1="30.48" x2="342.9" y2="33.02" width="0.1524" layer="91"/>
 <label x="335.28" y="17.78" size="1.778" layer="95" rot="R90"/>
 </segment>
