File: Eagle-Board/bike_tracker.sch (EAGLE design)
At the start: 93 parts, among them IC1 24C00TS, IC2 BME280/680, J1 TRANSFLASH-LOCK, Q1 IRLML5203, Q2 IRLML5203, Q3 IRLML5203, Q4 IRLML5203, U1 MPU-9250/5

Commit message: wireless charging option added
Parts:
- added C29, C30: 22nF, resistor:C-EUC0603
- added C31, C32: 0.47uF, resistor:C-EUC0603
- added C33, C34: 0.01uF, resistor:C-EUC0603
- added C35: 100pF, resistor:C-EUC0603
- added C36: 1800pF, resistor:C-EUC0603
- added C37: 47nF, resistor:C-EUC0603
- added C38, C39: 68nF, resistor:C-EUC0603
- added C40, C41: 10uF, sparkfun:CAP1206
- added C42, C44, C45: 0.1uF, resistor:C-EUC0603
- added C43: 1.0uF, resistor:C-EUC0603
- added COIL: 332-02, con-garry:332-02
- added D2: MBR0520, microduino:DIODE-SOD123
- added R48: 196, resistor:R-EU_R0603
- added R49: 75, resistor:R-EU_R0603
- added R50, R52, R53: 1.5k, resistor:R-EU_R0603
- added R51: 20k, resistor:R-EU_R0603
- added R54: 10k NTC, resistor:R-EU_R0603
- added U$3: BQ51013BQFN-20, WirelessPower:BQ51013BQFN-20
- added WIR.CH.: (no value), led:LEDSML0805
- U1: value MPU-9250/5 -> IMU9250
Connections:
- new net 5V: D2.C, ESP32-LORA.5V@35
- new net AC1: C29.2, C31.1, C33.1, C35.1, C36.1, C37.2, C38.2, C39.2, U$3.AC1
- new net AC1'1: C37.1, C38.1, C39.1, COIL-1.S
- new net AC2: C30.1, C32.1, C34.1, C35.2, C36.2, COIL-2.S, U$3.AC2
- new net BOOT1: C33.2, U$3.BOOT1
- new net BOOT2: C34.2, U$3.BOOT2
- new net CHG: U$3./WPG, WIR.CH..C
- new net CLMP1: C31.2, U$3.CLAMP1
- new net CLMP2: C32.2, U$3.CLAMP2
- new net COMM1: C29.1, U$3.COMM1
- new net COMM2: C30.2, U$3.COMM2
- new net FOD: C45.1, R48.2, R49.1, R51.1, U$3.FOD
- new net ILIM: R49.2, U$3.ILIM
- new net N$30: R50.1, WIR.CH..A
- new net N$31: R52.1, R54.2
- new net N$32: R53.1, R54.1
- new net OUT: C43.1, C44.1, D2.A, U$3.OUT
- new net RECT: C40.1, C41.1, C42.1, R50.2, R51.2, U$3.RECT
- new net TS-CTRL: R52.2, R53.2, U$3.TS-CTRL
- net GND: now also C40.2, C41.2, C42.2, C43.2, C44.2, C45.2, R48.1, U$3.AD, U$3.EN1/TERM, U$3.EN2, U$3.PGND

Commit message: added compatibility with TTGO LoRa v2.0
Parts:
- added R38, R39, R43, R44: 0, resistor:R-EU_R0603
- added R45: 1M, resistor:R-EU_R0603
- added R46, R47, R55, R56, R57, R58, R59, R60, R62, R63, R64, R65: (no value), resistor:R-EU_R0201
Connections:
- removed net 5V: D2.C, ESP32-LORA.5V@35
- removed net IO25: ESP32-LORA.IO25, R90.2
- new net 5V+: D2.C, ESP32-LORA.5V/X, R46.2, R58.1
- new net IO22: ESP32-LORA.IO22/14, R90.2
- new net N$28: R38.2, R48.1
- new net N$29: R39.2, R51.1
- new net N$36: R38.1, R43.2
- new net N$37: R39.1, R44.2
- new net N$38: ESP32-LORA.IO15/35, R47.1
- new net N$39: ESP32-LORA.IO04/RST, R55.1
- new net N$40: ESP32-LORA.IO14/22, R57.1
- new net N$41: ESP32-LORA.IO34/05, R59.1
- new net N$42: ESP32-LORA.IO16/36, R60.2
- new net N$43: ESP32-LORA.3V3/IO00, R62.1
- new net N$45: ESP32-LORA.5V/3.3, R63.1, R65.1
- new net N$46: ESP32-LORA.IO35/18, R64.1
- net FOD: now also R44.1; no longer R51.1
- net GND: now also ESP32-LORA.GND@/X, R43.1, R45.2, R53.1, R54.1; no longer ESP32-LORA.GND@1, R48.1, U$3.AD
- net INT-IMU: now also ESP32-LORA.IO36/04; no longer ESP32-LORA.IO36
- net IO26: now also ESP32-LORA.IO26/D12; no longer ESP32-LORA.IO26
- net IO32: now also ESP32-LORA.IO32/23; no longer ESP32-LORA.IO32
- net IO33: now also ESP32-LORA.IO33/26; no longer ESP32-LORA.IO33
- net IO35: now also R63.2, R64.2; no longer ESP32-LORA.IO35
- net IO37: now also ESP32-LORA.IO37/02; no longer ESP32-LORA.IO37
- net IO38: now also ESP32-LORA.IO38/15; no longer ESP32-LORA.IO38
- net IO39: now also ESP32-LORA.IO39/13; no longer ESP32-LORA.IO39
- net N$12: now also ESP32-LORA.IO01/5V, R58.2; no longer ESP32-LORA.IO05
- net N$32: now also R45.1, R46.1, U$3.AD; no longer R53.1, R54.1
- net RX: now also R59.2, R60.1; no longer ESP32-LORA.IO34
- net SCL: now also R47.2, R56.2; no longer ESP32-LORA.IO15
- net SDA: now also R55.2, R57.2; no longer ESP32-LORA.IO04
- net SPI-CLK: now also ESP32-LORA.IO23/25; no longer ESP32-LORA.IO23
- net SPI-CS: now also R56.1
- net SPI-MISO: now also ESP32-LORA.IO12/03; no longer ESP32-LORA.IO12
- net SPI-MOSI: now also ESP32-LORA.IO13/01; no longer ESP32-LORA.IO13
- net TX: now also ESP32-LORA.IO17/39; no longer ESP32-LORA.IO17
- net VDD: now also ESP32-LORA.3V3/X, R62.2, R65.2; no longer ESP32-LORA.3V3@3, ESP32-LORA.3V3@34
Other:
- moved on the sheet: C29, C30, C31, C32, C33, C34, C45, D, IC1, JP3, L, Q1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

Commit message: minor error correction and exported for production!
Parts:
- added C12: 1uF, resistor:C-EUC0603
- added R61, R66: (no value), resistor:R-EU_R0201
- C40, C41: device sparkfun:CAP1206 -> resistor:C-EUC0603
Connections:
- removed net IO26: ESP32-LORA.IO26/D12, R19.2
- removed net IO32: ESP32-LORA.IO32/23, R23.2
- removed net IO33: ESP32-LORA.IO33/26, R21.2
- new net IO25: ESP32-LORA.IO25/D11, R19.2
- new net N$44: ESP32-LORA.IO00/12, R61.2
- new net N$47: ESP32-LORA.IO22/14, R66.2
- new net N$48: ESP32-LORA.IO32/23, R63.1
- net GND: now also C12.1, ESP32-LORA.GND/X@1
- net IO22: now also R61.1, R66.1; no longer ESP32-LORA.IO22/14
- net IO35: now also R21.2
- net IO39: now also R23.2
- net N$32: now also C12.2
- net N$45: no longer R63.1
- net VBAT+: now also BAT-IN-1.S; no longer BAT-IN-2.S
- net VBAT-: now also BAT-IN-2.S; no longer BAT-IN-1.S
Other:
- moved on the sheet: C40, C41, R45, R46, R62, R63, U$3
